File: hardware/connectors.kicad_sch (KiCad schematic)
At the start: 24 parts, among them J1 USB-309GC-B-SU, J12 Conn_01x05, J8 Conn_01x03, U5 MAX17502EATB+T

Commit message: Ready for trial submit to JLCPCB
Connections:
- net GND: now also J12.5 (Pin_5); no longer J12.1 (Pin_1)
- net at C3.1, C61.1, C65.1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: now also J12.4 (Pin_4); no longer J12.2 (Pin_2)
- net at D7.2 (A): now also J12.2 (Pin_2); no longer J12.4 (Pin_4)
- net at D6.2 (A): now also J12.1 (Pin_1); no longer J12.5 (Pin_5)
Other:
- moved on the sheet: J12
Changed lines of the file:
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@@
+		)
+	)
+	(netclass_flag ""
+		(length 2.54)
+		(shape round)
+		(at 111.76 30.48 0)
+		(fields_autoplaced yes)
+		(effects
+			(font
+				(size 1.27 1.27)
+			)
+			(justify left bottom)
+		)
+		(property "Netclass" "HV"
+			(at 112.4585 27.94 0)
+			(effects
+				(font
+					(size 1.27 1.27)
+					(italic yes)
+				)
+				(justify left)
+			)
+		)
+	)
+	(netclass_flag ""
+		(length 2.54)
+		(shape round)
+		(at 111.76 38.1 0)
+		(fields_autoplaced yes)
+		(effects
+			(font
+				(size 1.27 1.27)
+			)
+			(justify left bottom)
+		)
+		(property "Netclass" "HV"
+			(at 112.4585 35.56 0)
+			(effects
+				(font
+					(size 1.27 1.27)
+					(italic yes)
+				)
+				(justify left)
+			)
+		)
+	)
+	(netclass_flag ""
+		(length 2.54)
+		(shape round)
+		(at 111.76 45.72 0)
+		(fields_autoplaced yes)
+		(effects
+			(font
+				(size 1.27 1.27)
+			)
+			(justify left bottom)
+		)
+		(property "Netclass" "HV"
+			(at 112.4585 43.18 0)
+			(effects
+				(font
+					(size 1.27 1.27)
+					(italic yes)
+				)
+				(justify left)
+			)
 		)
 	)
@@
 	(symbol
 		(lib_id "Connector_Generic:Conn_01x05")
-		(at 92.71 45.72 180)
+		(at 92.71 45.72 0)
+		(mirror y)
 		(unit 1)
 		(exclude_from_sim no)
@@
 		(on_board yes)
 		(dnp no)
-		(fields_autoplaced yes)
 		(property "Reference" "J12"
-			(at 92.71 34.29 0)
+			(at 92.71 57.15 0)
 			(effects
 				(font
@@
 		)
 		(property "Value" "Conn_01x05"
-			(at 92.71 36.83 0)
-			(effects
-				(font
+			(at 92.71 54.61 0)
+			(effects
+				(font

Commit message: * Added the JLCPCB Fabrication Plugin into KiCad and use this for the exports * Fixed problem detected with capacitor footprint for C42, C43, C44, C50, C51, C52
Parts:
- C3, C61: LCSC Part (none) -> C13832
- C5, C62: LCSC Part (none) -> C15850
- C63: LCSC Part (none) -> C1779
- C64: LCSC Part (none) -> C1613
- C65: LCSC Part (none) -> C128515
- D14: LCSC Part (none) -> C2286
- D5, D6, D7, D8: LCSC Part (none) -> C3758930
- L3: LCSC Part (none) -> C83472
- R51, R52: LCSC Part (none) -> C23186
- R57: LCSC Part (none) -> C21190
- U5: LCSC Part C559500 -> C571005
Changed lines of the file:
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@@
 			)
 		)
+		(property "LCSC Part" "C3758930"
+			(at 119.38 38.1 0)
+			(effects
+				(font
+					(size 1.27 1.27)
+				)
+				(hide yes)
+			)
+		)
 		(pin "1"
 		)
@@
 			)
 		)
+		(property "LCSC Part" "C2286"
+			(at 256.54 73.66 0)
+			(effects
+				(font
+					(size 1.27 1.27)
+				)
+				(hide yes)
+			)
+		)
 		(pin "1"
 		)
@@
 			)
 		)
+		(property "LCSC Part" "C1779"
+			(at 166.37 69.85 0)
+			(effects
+				(font
+					(size 1.27 1.27)
+				)
+				(hide yes)
+			)
+		)
 		(pin "2"
 		)
@@
 			)
 		)
+		(property "LCSC Part" "C23186"
+			(at 49.53 107.95 0)
+			(effects
+				(font
+					(size 1.27 1.27)
+				)
+				(hide yes)
+			)
+		)
 		(pin "2"
 		)
@@
 			)
 		)
+		(property "LCSC Part" "C83472"
+			(at 227.33 58.42 0)
+			(effects
+				(font
+					(size 1.27 1.27)
+				)
+				(hide yes)
+			)
+		)
 		(pin "1"
 		)
@@
 			)
 		)
+		(property "LCSC Part" "C15850"
+			(at 240.03 72.39 0)
+			(effects
+				(font
+					(size 1.27 1.27)
+				)
+				(hide yes)
+			)
+		)
 		(pin "1"
 		)
@@
 			)
 		)
+		(property "LCSC Part" "C15850"
+			(at 232.41 72.39 0)
+			(effects
+				(font
+					(size 1.27 1.27)
+				)
+				(hide yes)
+			)
+		)
 		(pin "1"
 		)
@@
 			)
 		)
+		(property "LCSC Part" "C23186"
+			(at 96.52 107.95 0)
+			(effects
+				(font
+					(size 1.27 1.27)
+				)
+				(hide yes)
+			)
+		)
 		(pin "2"
 		)
@@
 			)
 		)
+		(property "LCSC Part" "C21190"
+			(at 256.54 63.5 0)
+			(effects
+				(font
+					(size 1.27 1.27)
+				)
+				(hide yes)
+			)
+		)
 		(pin "1"
 		)
@@
 			)
 		)
+		(property "LCSC Part" "C1613"
+			(at 215.9 72.39 0)
+			(effects
+				(font
+					(size 1.27 1.27)
+				)
+				(hide yes)
+			)
+		)
 		(pin "2"
 		)
@@
 			)
 		)
+		(property "LCSC Part" "C13832"
+			(at 156.21 69.85 0)
+			(effects
+				(font
+					(size 1.27 1.27)
+				)
+				(hide yes)
+			)
+		)
 		(pin "2"
 		)
@@
 			)
 		)
+		(property "LCSC Part" "C128515"
+			(at 135.89 69.85 0)
+			(effects
+				(font
+					(size 1.27 1.27)
+				)
+				(hide yes)
+			)
+		)
 		(pin "1"
 		)
@@
 			)
 		)
-		(property "LCSC Part" "C559500"
+		(property "LCSC Part" "C571005"
 			(at 195.58 81.28 0)
 			(effects
@@
 			)
 		)
+		(property "LCSC Part" "C3758930"
+			(at 119.38 60.96 0)
+			(effects
+				(font
+					(size 1.27 1.27)
+				)
+				(hide yes)
+			)
+		)
 		(pin "1"
 		)
@@
 			)
 		)
+		(property "LCSC Part" "C3758930"
+			(at 119.38 30.48 0)
+			(effects
+				(font
+					(size 1.27 1.27)
+				)
+				(hide yes)
+			)
+		)
 		(pin "1"
 		)
@@
 			)
 		)
+		(property "LCSC Part" "C13832"
+			(at 146.05 69.85 0)
+			(effects
+				(font
+					(size 1.27 1.27)
+				)
+				(hide yes)
+			)
+		)
 		(pin "2"
 		)
@@
 			(at 119.38 45.72 0)
 			(effects
+				(font
+					(size 1.27 1.27)
+				)
+				(hide yes)
+			)
+		)
+		(property "LCSC Part" "C3758930"
+			(at 119.38 45.72 0)
+			(effects
